File: NewPCB/opsx_x/opsx_x.kicad_pcb (KiCad board)
At the start: 2 copper layers, 95.9 x 27.8 mm, 23 parts, among them J1 Conn_01x02, U1 RP2040, U2 TLV70430DBVR, U3 W25Q128JVS

Commit message: work
Parts:
- added D1: 1N4148WS, Diode_SMD:D_SOD-323, F.Cu at (40.1, 84.0)
- added D2: SFH2430, OptoDevice:Osram_SFH2430, B.Cu at (41.6, 65.8)
- added D3: 1N4148WS, Diode_SMD:D_SOD-323, F.Cu at (108.0, 78.6)
- added D4: 1N4148WS, Diode_SMD:D_SOD-323, F.Cu at (106.8, 61.8)
- added J2: Conn_01x02, Connector_PinHeader_2.54mm:PinHeader_1x02_P2.54mm_Vertical, F.Cu at (27.1, 78.0)
- added J3: Conn_01x02, Connector_PinHeader_2.54mm:PinHeader_1x02_P2.54mm_Vertical, F.Cu at (51.6, 74.2)
- added Q1: Q_NMOS_GSD, Package_TO_SOT_SMD:SOT-23, F.Cu at (108.0, 76.0)
- added Q2: Q_NMOS_GSD, Package_TO_SOT_SMD:SOT-23, F.Cu at (110.7, 60.6)
- added R10: 120, Resistor_SMD:R_0402_1005Metric_Pad0.72x0.64mm_HandSolder, F.Cu at (48.0, 65.4)
- added R11: 10k, Resistor_SMD:R_0402_1005Metric_Pad0.72x0.64mm_HandSolder, F.Cu at (38.6, 62.7)
- added R12: 10k, Resistor_SMD:R_0402_1005Metric_Pad0.72x0.64mm_HandSolder, F.Cu at (38.6, 63.7)
- added R13: 100, Resistor_SMD:R_0402_1005Metric_Pad0.72x0.64mm_HandSolder, F.Cu at (99.4, 68.6)
- added R14: 120, Resistor_SMD:R_0402_1005Metric_Pad0.72x0.64mm_HandSolder, F.Cu at (99.4, 70.9)
- added R15: 100, Resistor_SMD:R_0402_1005Metric_Pad0.72x0.64mm_HandSolder, F.Cu at (100.4, 69.0)
- added R16: 120, Resistor_SMD:R_0402_1005Metric_Pad0.72x0.64mm_HandSolder, F.Cu at (100.4, 71.3)
- added R17: 100, Resistor_SMD:R_0402_1005Metric_Pad0.72x0.64mm_HandSolder, F.Cu at (107.8, 69.5)
- added R18: 120, Resistor_SMD:R_0402_1005Metric_Pad0.72x0.64mm_HandSolder, F.Cu at (107.8, 68.4)
- added R19: 100, Resistor_SMD:R_0402_1005Metric_Pad0.72x0.64mm_HandSolder, F.Cu at (107.8, 71.6)
- added R20: 120, Resistor_SMD:R_0402_1005Metric_Pad0.72x0.64mm_HandSolder, F.Cu at (107.8, 70.6)
- added R21: 100, Resistor_SMD:R_0402_1005Metric_Pad0.72x0.64mm_HandSolder, F.Cu at (112.9, 74.3)
- added R22: 100, Resistor_SMD:R_0402_1005Metric_Pad0.72x0.64mm_HandSolder, F.Cu at (104.5, 77.2)
- added R23: 100k, Resistor_SMD:R_0402_1005Metric_Pad0.72x0.64mm_HandSolder, F.Cu at (105.5, 76.8)
- added R24: 100, Resistor_SMD:R_0402_1005Metric_Pad0.72x0.64mm_HandSolder, F.Cu at (104.3, 64.2)
- added R25: 100k, Resistor_SMD:R_0402_1005Metric_Pad0.72x0.64mm_HandSolder, F.Cu at (105.3, 64.1)
- added R5: 120, Resistor_SMD:R_0402_1005Metric_Pad0.72x0.64mm_HandSolder, F.Cu at (36.1, 82.1)
- added R6: 100, Resistor_SMD:R_0402_1005Metric_Pad0.72x0.64mm_HandSolder, F.Cu at (36.1, 83.1)
- added R9: 100, Resistor_SMD:R_0402_1005Metric_Pad0.72x0.64mm_HandSolder, F.Cu at (49.0, 65.4)
- added U4: OPTICAL-TSL2561T(6P-3.8X2.6MM), OPSX:TMB6-1.55-3.8X2.6MM, B.Cu at (41.6, 65.8)
- added Y1: Crystal_GND2, Crystal:Resonator_SMD_Murata_CSTxExxV-3Pin_3.0x1.1mm, F.Cu at (47.1, 68.5)
- added Z1: ~, OPSX:Selector_default, B.Cu at (37.0, 69.6)
- added Z2: ~, OPSX:Selector_default, B.Cu at (103.0, 65.1)
- sx1: value ~ -> sx~; footprint 0JIMMY:SX70 -> OPSX:sx70
- moved C10 18.9 mm to (44.6, 64.8)
- moved C9 18.5 mm to (40.0, 77.3), turned to -90 degrees
- moved J1 17.9 mm to (55.2, 74.2), turned to 0 degrees
- moved C5 5.83 mm to (37.0, 76.7), turned to 180 degrees
- moved C14 5.22 mm to (27.4, 73.2), turned to 180 degrees
- moved C2 4.93 mm to (50.0, 65.4), turned to 90 degrees
- moved C12 3.64 mm to (29.4, 67.7), turned to 180 degrees
- moved C6 3.33 mm to (35.2, 66.6)
- moved C7 3.33 mm to (36.2, 66.7)
- moved C8 2.99 mm to (34.1, 66.6)
- moved C1 2.99 mm to (33.1, 66.6)
- moved R1 2.96 mm to (31.1, 66.6)
- moved R2 2.96 mm to (32.1, 66.6)
- moved C11 2.78 mm to (41.0, 77.3)
- moved C3 2.68 mm to (29.4, 68.7), turned to 180 degrees
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Connections:
- U1 pad 12: unconnected-(U1-GPIO9-Pad12) -> /SOL1_MCU
- U1 pad 13: unconnected-(U1-GPIO10-Pad13) -> /SDA1
- U1 pad 14: unconnected-(U1-GPIO11-Pad14) -> /SCL1
- U1 pad 15: unconnected-(U1-GPIO12-Pad15) -> /URAT0_TX
- U1 pad 16: unconnected-(U1-GPIO13-Pad16) -> /URAT0_RX
- U1 pad 2: unconnected-(U1-GPIO0-Pad2) -> /GTD-3
- U1 pad 20: unconnected-(U1-XIN-Pad20) -> /XIN
- U1 pad 21: unconnected-(U1-XOUT-Pad21) -> /XOUT
- U1 pad 28: unconnected-(U1-GPIO17-Pad28) -> /SOL2_MCU
- U1 pad 29: unconnected-(U1-GPIO18-Pad29) -> /FF
- U1 pad 3: unconnected-(U1-GPIO1-Pad3) -> /S1T-3
- U1 pad 30: unconnected-(U1-GPIO19-Pad30) -> /S2
- U1 pad 31: unconnected-(U1-GPIO20-Pad31) -> /SDA0
- U1 pad 32: unconnected-(U1-GPIO21-Pad32) -> /SCL0
- U1 pad 38: unconnected-(U1-GPIO26_ADC0-Pad38) -> /FT-3
- U1 pad 4: unconnected-(U1-GPIO2-Pad4) -> /S1F-3
- U1 pad 5: unconnected-(U1-GPIO3-Pad5) -> /S9-3
- U1 pad 6: unconnected-(U1-GPIO4-Pad6) -> /S8-3
- U1 pad 7: unconnected-(U1-GPIO5-Pad7) -> Net-(U1-GPIO5)
- U1 pad 8: unconnected-(U1-GPIO6-Pad8) -> /S5
- U1 pad 9: unconnected-(U1-GPIO7-Pad9) -> /S3
- sx1 pad F+: unconnected-(sx1-PadF+) -> +3.3V
- sx1 pad F-: unconnected-(sx1-PadF-) -> /S1T-3
- sx1 pad FF: unconnected-(sx1-PadFF) -> /FF
- sx1 pad FT: unconnected-(sx1-PadFT) -> /FT
- sx1 pad GND: unconnected-(sx1-PadGND) -> GND
- sx1 pad GTD: unconnected-(sx1-PadGTD) -> /GTD-6
- sx1 pad MOTOR: unconnected-(sx1-PadMOTOR) -> /MOTOR
- sx1 pad S1C: unconnected-(sx1-PadS1C) -> VCC
- sx1 pad S1F: unconnected-(sx1-PadS1F) -> /S1F
- sx1 pad S1T: unconnected-(sx1-PadS1T) -> /S1T
- sx1 pad S2: unconnected-(sx1-PadS2) -> /S2
- sx1 pad S2+: unconnected-(sx1-PadS2+) -> /S2
- sx1 pad S2-: (no net) -> GND
- sx1 pad S3: unconnected-(sx1-PadS3) -> /S3
- sx1 pad S5: unconnected-(sx1-PadS5) -> /S5
- sx1 pad S8: unconnected-(sx1-PadS8) -> /S8
- sx1 pad S9: unconnected-(sx1-PadS9) -> /S9
- sx1 pad SOL2+: unconnected-(sx1-PadSOL2+) -> VCC
- sx1 pad SOL2-: unconnected-(sx1-PadSOL2-) -> /SOL2-
- sx1 pad VCC: unconnected-(sx1-PadVCC) -> VCC
Routing:
- net /S1T-3: track 0.00 -> 129.5 mm, vias 0 -> 5
- net VCC: track 1.50 -> 123.9 mm, vias 0 -> 4
- net /S5: track 0.00 -> 86.8 mm, vias 0 -> 2
- net /S3: track 0.00 -> 85.6 mm, vias 0 -> 2
- net /S2: track 0.00 -> 83.4 mm, vias 0 -> 3
- net /S1F-3: track 0.00 -> 80.0 mm, vias 0 -> 4
- net /S9-3: track 0.00 -> 79.7 mm, vias 0 -> 4
- net Net-(U1-GPIO5): track 0.00 -> 79.4 mm, vias 0 -> 2
- net /S8-3: track 0.00 -> 78.0 mm, vias 0 -> 2
- net /SOL1_MCU: track 0.00 -> 69.6 mm, vias 0 -> 2
- net /GTD-6: track 0.00 -> 67.6 mm, vias 0 -> 2
- net /SOL2_MCU: track 0.00 -> 67.1 mm, vias 0 -> 2
- net /FF: track 0.00 -> 64.4 mm, vias 0 -> 2
- net /FT: track 0.00 -> 59.8 mm, vias 0 -> 2
- net GND: track 15.2 -> 47.9 mm, vias 15 -> 41
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- added copper zone on F.Cu, net GND
- added copper zone on F.Cu, net VCC
Other:
- board text added: "Connect to Flash Socket"
- board text added: "GND"
- board text added: "S2"
- board text added: "TSL_ADD"
- board text added: "USB BOOT"
- board text added: "V+"
- board text added: "locked"

Commit message: PCB  finished
finished pcb designing, god bless it would work.
Parts:
- added C15: 13p, Capacitor_SMD:C_0402_1005Metric_Pad0.74x0.62mm_HandSolder, F.Cu at (108.0, 67.8)
- added D5: LED, Diode_SMD:D_0603_1608Metric_Pad1.05x0.95mm_HandSolder, F.Cu at (53.3, 60.2)
- added D6: LED, Diode_SMD:D_0603_1608Metric_Pad1.05x0.95mm_HandSolder, F.Cu at (53.3, 58.7)
- added Q3: Q_PMOS_GSD, Package_TO_SOT_SMD:SOT-23, F.Cu at (108.5, 71.1)
- added Q4: MMBT3904, Package_TO_SOT_SMD:SOT-23, F.Cu at (90.5, 62.7)
- added R26: 1k, Resistor_SMD:R_0402_1005Metric_Pad0.72x0.64mm_HandSolder, F.Cu at (100.1, 70.3)
- added R27: 1k, Resistor_SMD:R_0402_1005Metric_Pad0.72x0.64mm_HandSolder, F.Cu at (102.8, 73.7)
- added R28: 100k, Resistor_SMD:R_0402_1005Metric_Pad0.72x0.64mm_HandSolder, F.Cu at (100.6, 76.5)
- added R29: 180, Resistor_SMD:R_0402_1005Metric_Pad0.72x0.64mm_HandSolder, F.Cu at (40.6, 82.5)
- added R30: 150, Resistor_SMD:R_0402_1005Metric_Pad0.72x0.64mm_HandSolder, F.Cu at (97.8, 80.8)
- added R31: 5.6k, Resistor_SMD:R_0402_1005Metric_Pad0.72x0.64mm_HandSolder, F.Cu at (93.7, 63.8)
- added R32: 47k, Resistor_SMD:R_0402_1005Metric_Pad0.72x0.64mm_HandSolder, F.Cu at (88.6, 60.7)
- added R33: 2.7k, Resistor_SMD:R_0402_1005Metric_Pad0.72x0.64mm_HandSolder, F.Cu at (102.6, 64.3)
- added R34: 330, Resistor_SMD:R_0402_1005Metric_Pad0.72x0.64mm_HandSolder, F.Cu at (36.3, 63.8)
- added R35: 1k, Resistor_SMD:R_0402_1005Metric_Pad0.72x0.64mm_HandSolder, F.Cu at (46.3, 71.0)
- added R7: 22k, Resistor_SMD:R_0805_2012Metric_Pad1.20x1.40mm_HandSolder, F.Cu at (105.7, 69.3)
- added R8: 100k, Resistor_SMD:R_0402_1005Metric_Pad0.72x0.64mm_HandSolder, F.Cu at (98.0, 73.9)
- added U5: AD8603, Package_TO_SOT_SMD:TSOT-23-5, F.Cu at (102.9, 69.1)
- added U6: AD8603, Package_TO_SOT_SMD:TSOT-23-5, F.Cu at (100.4, 73.9)
- added Z3: ~, OPSX:Selector_default, B.Cu at (97.0, 65.6)
- R10, R14, R16, R18, R20, R5: value 120 -> 12k
- R13, R15, R17, R19, R6, R9: value 100 -> 10k
- moved R18 11.6 mm to (119.4, 69.6), turned to -90 degrees
- moved R20 10.6 mm to (118.4, 70.1), turned to 90 degrees
- moved R17 9.87 mm to (117.6, 68.3), turned to 0 degrees
- moved R19 9.65 mm to (117.3, 70.1), turned to -90 degrees
- moved C7 8.65 mm to (35.2, 75.3), turned to -90 degrees
- moved C13 8.62 mm to (36.2, 66.6), turned to 90 degrees
- moved R16 4.92 mm to (95.5, 70.9)
- moved C6 4.16 mm to (31.0, 66.5)
- moved R15 3.38 mm to (97.0, 68.8), turned to 180 degrees
- moved R14 3.20 mm to (98.6, 67.8), turned to 0 degrees
- moved R2 2.28 mm to (34.2, 67.5)
- moved R1 2.28 mm to (33.2, 67.5)
- moved C1 2.24 mm to (35.2, 67.4)
- moved C8 2.08 mm to (32.0, 66.5)
- moved R13 1.99 mm to (98.6, 66.8), turned to 180 degrees
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Connections:
- D2 pad 1: unconnected-(D2-K-Pad1) -> Net-(D2-K)
- D2 pad 2: unconnected-(D2-A-Pad2) -> GND
- U1 pad 13: /SDA1 -> unconnected-(U1-GPIO10-Pad13)
- U1 pad 14: /SCL1 -> /S4A_3
- U1 pad 15: /URAT0_TX -> /LED2
- U1 pad 16: /URAT0_RX -> /LED1
- U1 pad 21: /XOUT -> Net-(U1-XOUT)
- U1 pad 34: unconnected-(U1-GPIO22-Pad34) -> /S1F_PF_MCU
- U1 pad 39: unconnected-(U1-GPIO27_ADC1-Pad39) -> /SFH_H
- U1 pad 40: unconnected-(U1-GPIO28_ADC2-Pad40) -> /SFH_L
- Z2 pad 1: /S1F_PF -> /S1F
- Z2 pad 3: /S1F -> /S1F_FPC
- sx1 pad F-: /S1T-3 -> /S1T
- sx1 pad S4A: unconnected-(sx1-PadS4A) -> /S4A_3
- sx1 pad S4B: unconnected-(sx1-PadS4B) -> /S4B
Routing:
- net /SFH_H: track 0.00 -> 87.0 mm, vias 0 -> 4
- net Net-(D2-K): track 0.00 -> 82.5 mm, vias 0 -> 1
- net +3.3V: track 55.6 -> 132.3 mm, vias 5 -> 7
- net /S4A_3: track 0.00 -> 74.6 mm, vias 0 -> 3
- net /SFH_L: track 0.00 -> 73.7 mm, vias 0 -> 4
- net /S1F_PF_MCU: track 0.00 -> 59.9 mm, vias 0 -> 4
- net /S1T: track 28.4 -> 84.7 mm, vias 0 -> 2
- net /S1T-3: track 129.5 -> 77.3 mm, vias 5 -> 4
- net GND: track 47.9 -> 85.5 mm, vias 41 -> 57
- net Net-(Q3-G): track 0.00 -> 35.8 mm, vias 0 -> 4
- net /LED2: track 0.00 -> 25.6 mm, vias 0 -> 2
- net /LED1: track 0.00 -> 23.2 mm, vias 0 -> 2
- net Net-(D5-A): track 0.00 -> 20.1 mm, vias 0 -> 2
- net /S8-3: track 78.0 -> 97.0 mm
- net VCC: track 123.9 -> 141.9 mm, vias 4 -> 6
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- added copper zone on F.Cu, net /SOL2-
