File: NewPCB/opsx_x/opsx_x.kicad_sch (KiCad schematic)
At the start: 23 parts, among them J1 Conn_01x02, U1 RP2040, U2 TLV70430DBVR, U3 W25Q128JVS

Commit message: work
Parts:
- added D1, D3, D4: 1N4148WS, Diode_SMD:D_SOD-323, symbol Diode:1N4148WS
- added D2: SFH2430, OptoDevice:Osram_SFH2430, symbol Sensor_Optical:SFH2430
- added J2, J3: Conn_01x02, Connector_PinHeader_2.54mm:PinHeader_1x02_P2.54mm_Vertical, symbol Connector_Generic:Conn_01x02
- added Q1, Q2: Q_NMOS_GSD, Package_TO_SOT_SMD:SOT-23, symbol Device:Q_NMOS_GSD
- added R10, R14, R16, R18, R20, R5: 120, Resistor_SMD:R_0402_1005Metric_Pad0.72x0.64mm_HandSolder, symbol Device:R
- added R11, R12: 10k, Resistor_SMD:R_0402_1005Metric_Pad0.72x0.64mm_HandSolder, symbol Device:R
- added R13, R15, R17, R19, R21, R22, R24, R6, R9: 100, Resistor_SMD:R_0402_1005Metric_Pad0.72x0.64mm_HandSolder, symbol Device:R
- added R23, R25: 100k, Resistor_SMD:R_0402_1005Metric_Pad0.72x0.64mm_HandSolder, symbol Device:R
- added U4: OPTICAL-TSL2561T(6P-3.8X2.6MM), TMB6-1.55-3.8X2.6MM, symbol OPTICAL-TSL2561T_6P-3.8X2.6MM_:OPTICAL-TSL2561T(6P-3.8X2.6MM)
- added Y1: Crystal_GND2, Crystal:Resonator_SMD_Murata_CSTxExxV-3Pin_3.0x1.1mm, symbol Device:Crystal_GND2
- added Z1, Z2: ~, OPSX:Selector_default, symbol OPSX:selector_default
- sx1: value ~ -> sx~; footprint 0JIMMY:SX70 -> OPSX:sx70; symbol 0JIMMY:sx70 -> OPSX:sx70
Connections:
- net +3.3V: now also sx1.F+, R11.1, R12.1, U4.1 (VDD), Z1.1
- net GND: now also sx1.GND, sx1.S2-, J3.1 (Pin_1), Q1.2 (S), Q2.2 (S), R10.2, R14.2, R16.2, R18.2, R20.2, R23.1, R25.1, R5.2, U4.2 (ADDR), U4.3 (GND), Y1.2, Z1.2, Z1.3
- net USB_D+: now also J2.2 (Pin_2)
- net USB_D-: now also J2.1 (Pin_1)
- net VCC: now also sx1.S1C, sx1.SOL1+, sx1.SOL2+, sx1.VCC, D1.1 (K), D3.1 (K), D4.1 (K)
- net SOL1_MCU: now reaches U1.12 (GPIO9)
- net SOL1_MCU: now also R22.1
- net SDA1: now reaches U1.13 (GPIO10)
- net SCL1: now reaches U1.14 (GPIO11)
- net URAT0_TX: now reaches U1.15 (GPIO12)
- net URAT0_RX: now reaches U1.16 (GPIO13)
- net GTD-3: now reaches U1.2 (GPIO0)
- net GTD-3: now also R5.1, R6.2
- net XIN: now reaches U1.20 (XIN)
- net XIN: now also Y1.3
- net XOUT: now reaches U1.21 (XOUT)
- net XOUT: now also Y1.1
- net SOL2_MCU: now reaches U1.28 (GPIO17)
- net SOL2_MCU: now also R24.1
- net FF: now reaches U1.29 (GPIO18)
- net FF: now also sx1.FF
- net S1T-3: now reaches U1.3 (GPIO1)
- net S1T-3: now also sx1.F-, R13.2, R14.1
- net S2: now reaches U1.30 (GPIO19)
- net S2: now also sx1.S2, sx1.S2+
- net SDA0: now reaches U1.31 (GPIO20)
- net SDA0: now also R11.2, U4.6 (SDA)
- net SCL0: now reaches U1.32 (GPIO21)
- net SCL0: now also R12.2, U4.4 (SCL)
- net FT-3: now reaches U1.38 (GPIO26_ADC0)
- net FT-3: now also R10.1, R9.2
- net S1F-3: now reaches U1.4 (GPIO2)
- net S1F-3: now also R15.2, R16.1
- net S9-3: now reaches U1.5 (GPIO3)
- net S9-3: now also R19.2, R20.1
- net S8-3: now reaches U1.6 (GPIO4)
- net S8-3: now also R17.2, R18.1
- net at U1.7 (GPIO5): now also R21.1
- net S5: now reaches U1.8 (GPIO6)
- net S5: now also sx1.S5
- net S3: now reaches U1.9 (GPIO7)
- net S3: now also sx1.S3
- net FT: now reaches sx1.FT
- net FT: now also R9.1
- net GTD-6: now reaches sx1.GTD
- net GTD-6: now also R6.1
- net MOTOR: now reaches sx1.MOTOR
- net MOTOR: now also R21.2
- net S1F: now reaches sx1.S1F
- net S1F: now also R15.1, Z2.3
- net S1T: now reaches sx1.S1T
- net S1T: now also R13.1
- net S8: now reaches sx1.S8
- net S8: now also R17.1
- net S9: now reaches sx1.S9
- net S9: now also R19.1
- net SOL2-: now reaches sx1.SOL2-
- net SOL2-: now also D4.2 (A), Q2.3 (D)
- new net: Q1.1 (G), R22.2, R23.2
- new net: Q2.1 (G), R24.2, R25.2
- new net S1F_FPC: Z2.2, sx1.S1F_FPC
- new net S1F_PF: Z2.1
- new net SOL1-: D3.2 (A), Q1.3 (D), sx1.SOL1-
- new net VBUS: D1.2 (A), J3.2 (Pin_2)
- no-connect marks 2 -> 6
Other:
- note added: "Controller (RP2040 )"
- note added: "Crystal"
- note added: "Flash"
- note added: "IF Sonar: high means button got pressed ELSE : low"
- note added: "Meter0"
- note added: "Power"
- note added: "USB"
- note removed: "RP2040 as controller"
- moved on the sheet: C1, C14, C2, C4, C5, J1, R3, R4, U2, U3

Commit message: PCB  finished
finished pcb designing, god bless it would work.
Parts:
- added C15: 13p, Capacitor_SMD:C_0402_1005Metric_Pad0.74x0.62mm_HandSolder, symbol Device:C
- added D5, D6: LED, Diode_SMD:D_0603_1608Metric_Pad1.05x0.95mm_HandSolder, symbol Device:LED
- added Q3: Q_PMOS_GSD, Package_TO_SOT_SMD:SOT-23, symbol Device:Q_PMOS_GSD
- added Q4: MMBT3904, Package_TO_SOT_SMD:SOT-23, symbol Transistor_BJT:MMBT3904
- added R26, R27, R35: 1k, Resistor_SMD:R_0402_1005Metric_Pad0.72x0.64mm_HandSolder, symbol Device:R
- added R28, R8: 100k, Resistor_SMD:R_0402_1005Metric_Pad0.72x0.64mm_HandSolder, symbol Device:R
- added R29: 180, Resistor_SMD:R_0402_1005Metric_Pad0.72x0.64mm_HandSolder, symbol Device:R
- added R30: 150, Resistor_SMD:R_0402_1005Metric_Pad0.72x0.64mm_HandSolder, symbol Device:R
- added R31: 5.6k, Resistor_SMD:R_0402_1005Metric_Pad0.72x0.64mm_HandSolder, symbol Device:R
- added R32: 47k, Resistor_SMD:R_0402_1005Metric_Pad0.72x0.64mm_HandSolder, symbol Device:R
- added R33: 2.7k, Resistor_SMD:R_0402_1005Metric_Pad0.72x0.64mm_HandSolder, symbol Device:R
- added R34: 330, Resistor_SMD:R_0402_1005Metric_Pad0.72x0.64mm_HandSolder, symbol Device:R
- added R7: 22k, Resistor_SMD:R_0805_2012Metric_Pad1.20x1.40mm_HandSolder, symbol Device:R
- added U5, U6: AD8603, Package_TO_SOT_SMD:TSOT-23-5, symbol Amplifier_Operational:AD8603
- added Z3: ~, OPSX:Selector_default, symbol OPSX:selector_default
- R10, R14, R16, R18, R20, R5: value 120 -> 12k
- R13, R15, R17, R19, R6, R9: value 100 -> 10k
- R21, R22, R24: value 100 -> 120
Connections:
- net S1F_PF is gone; now on net S1F: Z2.1
- net SCL1 is gone; now on net S4A_3: U1.14 (GPIO11)
- net +3.3V: now also R34.2, U5.5 (V+), U6.5 (V+)
- net GND: now also D2.2 (A), Q4.2 (E), R26.1, R28.2, R29.2, R33.1, U5.2 (V-), U5.3 (+), U6.2 (V-)
- net S1F: no longer Z2.3
- net S1F_FPC: now also Z2.3, Q3.3 (D), R33.2
- net S1T: now also sx1.F-, Z3.2, Z3.3
- net S1T-3: now also Z3.1; no longer sx1.F-
- net VCC: now also Q3.2 (S), R32.1
- net XOUT: now also R35.1; no longer U1.21 (XOUT)
- net S1F_PF_MCU: now reaches U1.34 (GPIO22)
- net S1F_PF_MCU: now also R31.2
- net SFH_H: now reaches U1.39 (GPIO27_ADC1)
- net SFH_H: now also C15.2, R27.1, R7.2, U5.1
- net SFH_L: now reaches U1.40 (GPIO28_ADC2)
- net SFH_L: now also R8.2, U6.1
- net at D2.1 (K): now also C15.1, R7.1, U5.4 (-)
- net S4A_3: now reaches sx1.S4A
- net S4A_3: now also R29.1, R30.2
- net S4B: now reaches sx1.S4B
- net S4B: now also R30.1
- net SDA1: no longer names the net of U1.13 (GPIO10)
- net URAT0_RX renamed LED1
- net LED1: now also D5.1 (K)
- net URAT0_TX renamed LED2
- net LED2: now also D6.1 (K)
- new net: R35.2, U1.21 (XOUT)
- new net: R27.2, R28.1, U6.3 (+)
- new net: R26.2, R8.1, U6.4 (-)
- new net: Q4.1 (B), R31.1
- new net: Q3.1 (G), Q4.3 (C), R32.2
- new net: D5.2 (A), D6.2 (A), R34.1
- no-connect marks 6 -> 15
Other:
- note added: "Meter1"
- note added: "SCL1"
- note added: "SDA1"
- moved on the sheet: C14, D2, J1, R11, R12, R3, R4, U3, U4, Z1, Z2
