File: Sonnar/Body_controller/Rev1/Controller_body/Controller_body.kicad_pcb (KiCad board)
At the start: 2 copper layers, 40.6 x 79 mm, 22 parts, among them J1 Conn_01x06_Socket, U1 PCF8575PWR

Commit message: controller finished
Parts:
- added J2: Conn_01x03_Socket, Connector_PinHeader_2.54mm:PinHeader_1x03_P2.54mm_Horizontal, F.Cu at (113.7, 112.0)
Routing:
- net /UD+: track 0.00 -> 68.0 mm, vias 0 -> 1
- net /UD-: track 0.00 -> 67.2 mm, vias 0 -> 1
- net /M_1: track 16.9 -> 18.1 mm
- net /A_8: track 48.3 -> 47.2 mm
- net /A_4: track 46.2 -> 45.2 mm
- net /SCL: track 65.4 -> 64.5 mm
- net /SW_A: track 37.1 -> 37.7 mm
- net /M_2: track 15.3 -> 15.9 mm
- net /SW_B: track 29.0 -> 29.6 mm
- net /SW_PUSH: track 33.0 -> 33.6 mm
- net GND: vias 37 -> 41
Other:
- board text added: "GND"
- board text added: "U+"
- board text added: "U-"
