File: Sonnar/Body_controller/Rev1/Controller_body/Controller_body.kicad_pcb (KiCad board)
At the start: 2 copper layers, 40.6 x 79 mm, 23 parts, among them J1 Conn_01x06_Socket, J2 Conn_01x03_Socket, U1 PCF8575PWR

Commit message: code upgrade
Routing:
- added copper zone on F.Cu, net /SW_B
Changed lines of the file:
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@@
+    )
+  )
+  (zone (net 23) (net_name "/SW_B") (layer "F.Cu") (hatch edge 0.5)
+    (priority 3)
+    (connect_pads (clearance 0.7))
+    (min_thickness 0.25) (filled_areas_thickness no)
+    (fill yes (thermal_gap 0.5) (thermal_bridge_width 0.5))
+    (polygon
+      (pts
+        (xy 91.3 118.6)
+        (xy 91 118.6)
+        (xy 90.4 119.4)
+        (xy 92 119.4)
+      )
     )
   )

Commit message: case refined
Routing:
- net /SW_A: track 37.7 -> 37.2 mm
- net GND: vias 41 -> 40
Other:
- board size 40.6 x 79 mm -> 40.6 x 91.2 mm
Changed lines of the file:
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@@
   (gr_arc locked (start 103.632 95.25) (mid 101.863781 72.548436) (end 101.346 49.784)
     (stroke (width 0.1) (type default)) (layer "Edge.Cuts"))
-  (gr_line locked (start 79.756 128.778) (end 120.396 128.778)
+  (gr_line locked (start 79.8 141) (end 120.4 141)
     (stroke (width 0.1) (type default)) (layer "Edge.Cuts"))
   (gr_line locked (start 101.346 49.784) (end 83.058 49.784)
     (stroke (width 0.1) (type default)) (layer "Edge.Cuts"))
-  (gr_line locked (start 120.396 128.778) (end 120.396 99.568)
+  (gr_line locked (start 120.4 141) (end 120.396 99.568)
     (stroke (width 0.1) (type default)) (layer "Edge.Cuts"))
-  (gr_line locked (start 79.756 53.086) (end 79.756 128.778)
+  (gr_line locked (start 79.756 53.086) (end 79.8 141)
     (stroke (width 0.1) (type default)) (layer "Edge.Cuts"))
   (gr_rect (start 79.042 48.922001) (end 176.832 146.458001)
@@
   (segment (start 90.83 108.07) (end 91.618 108.07) (width 0.254) (layer "F.Cu") (net 10))
   (segment (start 92.162 56.388) (end 92.162 58.26) (width 0.254) (layer "F.Cu") (net 10))
-  (via (at 108.458 120.65) (size 0.8) (drill 0.4) (layers "F.Cu" "B.Cu") (free) (net 10))
+  (via (at 108.4 120.9) (size 0.8) (drill 0.4) (layers "F.Cu" "B.Cu") (free) (net 10))
   (via (at 108.458 125.73) (size 0.8) (drill 0.4) (layers "F.Cu" "B.Cu") (free) (net 10))
   (via (at 96.52 68.834) (size 0.8) (drill 0.4) (layers "F.Cu" "B.Cu") (free) (net 10))
@@
   (via (at 87.122 52.324) (size 0.8) (drill 0.4) (layers "F.Cu" "B.Cu") (free) (net 10))
   (via (at 97.79 117.856) (size 0.8) (drill 0.4) (layers "F.Cu" "B.Cu") (free) (net 10))
-  (via (at 86.868 126.492) (size 0.8) (drill 0.4) (layers "F.Cu" "B.Cu") (free) (net 10))
   (via (at 90.424 125.73) (size 0.8) (drill 0.4) (layers "F.Cu" "B.Cu") (free) (net 10))
   (via (at 96.52 75.946) (size 0.8) (drill 0.4) (layers "F.Cu" "B.Cu") (free) (net 10))
@@
   (via (at 88.646 114.3) (size 0.8) (drill 0.4) (layers "F.Cu" "B.Cu") (free) (net 10))
   (via (at 83.312 99.06) (size 0.8) (drill 0.4) (layers "F.Cu" "B.Cu") (free) (net 10))
-  (via (at 103.378 120.65) (size 0.8) (drill 0.4) (layers "F.Cu" "B.Cu") (free) (net 10))
+  (via (at 103.4 120.9) (size 0.8) (drill 0.4) (layers "F.Cu" "B.Cu") (free) (net 10))
   (via (at 90.2 109) (size 0.8) (drill 0.4) (layers "F.Cu" "B.Cu") (net 10))
   (via (at 99.568 114.3) (size 0.8) (drill 0.4) (layers "F.Cu" "B.Cu") (free) (net 10))
@@
   (via (at 96.52 79.502) (size 0.8) (drill 0.4) (layers "F.Cu" "B.Cu") (free) (net 10))
   (via (at 94.234 125.73) (size 0.8) (drill 0.4) (layers "F.Cu" "B.Cu") (free) (net 10))
-  (via (at 103.378 107.442) (size 0.8) (drill 0.4) (layers "F.Cu" "B.Cu") (free) (net 10))
+  (via (at 103.3 107.2) (size 0.8) (drill 0.4) (layers "F.Cu" "B.Cu") (free) (net 10))
   (via (at 98.806 125.73) (size 0.8) (drill 0.4) (layers "F.Cu" "B.Cu") (free) (net 10))
   (via (at 99.568 116.078) (size 0.8) (drill 0.4) (layers "F.Cu" "B.Cu") (free) (net 10))
@@
   (segment (start 87.436999 62.021999) (end 87.436999 66.673199) (width 0.2) (layer "B.Cu") (net 20))
   (segment (start 96.295 82.833) (end 96.295 92.739) (width 0.2) (layer "B.Cu") (net 20))
-  (segment (start 98.806 122.428) (end 95.504 122.428) (width 0.254) (layer "F.Cu") (net 21))
-  (segment (start 102.362 118.872) (end 98.806 122.428) (width 0.254) (layer "F.Cu") (net 21))
-  (segment (start 99.658 106.77) (end 102.362 109.474) (width 0.254) (layer "F.Cu") (net 21))
-  (segment (start 97.358 106.77) (end 99.658 106.77) (width 0.254) (layer "F.Cu") (net 21))
+  (segment (start 97.358 106.77) (end 98.97 106.77) (width 0.254) (layer "F.Cu") (net 21))
+  (segment (start 102.3 110.1) (end 102.3 118.8) (width 0.254) (layer "F.Cu") (net 21))
+  (segment (start 98.672 122.428) (end 95.504 122.428) (width 0.254) (layer "F.Cu") (net 21))
+  (segment (start 102.3 118.8) (end 98.672 122.428) (width 0.254) (layer "F.Cu") (net 21))
+  (segment (start 98.97 106.77) (end 102.3 110.1) (width 0.254) (layer "F.Cu") (net 21))
   (segment (start 95.504 122.428) (end 88.4915 122.428) (width 0.254) (layer "F.Cu") (net 21))
-  (segment (start 102.362 109.474) (end 102.362 118.872) (width 0.254) (layer "F.Cu") (net 21))
   (segment (start 95.25 117.078) (end 95.25 118.364) (width 0.254) (layer "F.Cu") (net 21))
   (segment (start 88.4915 122.428) (end 87.5155 123.404) (width 0.254) (layer "F.Cu") (net 21))
@@
   (segment (start 95.25 122.174) (end 95.504 122.428) (width 0.254) (layer "B.Cu") (net 21))
   (segment (start 93.98 120.904) (end 99.314 120.904) (width 0.254) (layer "F.Cu") (net 22))
-  (segment (start 99.314 120.904) (end 101.8 118.418) (width 0.254) (layer "F.Cu") (net 22))
+  (segment (start 98.72 107.42) (end 97.358 107.42) (width 0.254) (layer "F.Cu") (net 22))
+  (segment (start 99.314 120.904) (end 101.7 118.518) (width 0.254) (layer "F.Cu") (net 22))
+  (segment (start 101.7 110.4) (end 98.72 107.42) (width 0.254) (layer "F.Cu") (net 22))
   (segment (start 87.5155 120.904) (end 93.98 120.904) (width 0.254) (layer "F.Cu") (net 22))
   (segment (start 93.218 117.078) (end 93.218 118.364) (width 0.254) (layer "F.Cu") (net 22))
-  (segment (start 99.292 107.42) (end 97.358 107.42) (width 0.254) (layer "F.Cu") (net 22))
-  (segment (start 101.8 118.418) (end 101.8 109.928) (width 0.254) (layer "F.Cu") (net 22))
-  (segment (start 101.8 109.928) (end 99.292 107.42) (width 0.254) (layer "F.Cu") (net 22))
+  (segment (start 101.7 118.518) (end 101.7 110.4) (width 0.254) (layer "F.Cu") (net 22))
   (via (at 93.98 120.904) (size 0.8) (drill 0.4) (layers "F.Cu" "B.Cu") (net 22))
   (via (at 93.218 118.364) (size 0.8) (drill 0.4) (layers "F.Cu" "B.Cu") (net 22))
@@
   (segment (start 93.472 118.364) (end 93.218 118.364) (width 0.254) (layer "B.Cu") (net 22))
   (segment (start 93.98 120.904) (end 93.98 118.872) (width 0.254) (layer "B.Cu") (net 22))
-  (segment (start 91.948 119.38) (end 99.822 119.38) (width 0.254) (layer "F.Cu") (net 23))
-  (segment (start 101.092 110.236) (end 98.926 108.07) (width 0.254) (layer "F.Cu") (net 23))
+  (segment (start 98.47 108.07) (end 97.358 108.07) (width 0.254) (layer "F.Cu") (net 23))
+  (segment (start 101.092 110.692) (end 98.47 108.07) (width 0.254) (layer "F.Cu") (net 23))
   (segment (start 91.186 117.078) (end 91.186 118.618) (width 0.254) (layer "F.Cu") (net 23))
   (segment (start 91.186 118.618) (end 91.948 119.38) (width 0.254) (layer "F.Cu") (net 23))
-  (segment (start 101.092 118.11) (end 101.092 110.236) (width 0.254) (layer "F.Cu") (net 23))
+  (segment (start 91.948 119.38) (end 99.971 119.38) (width 0.254) (layer "F.Cu") (net 23))
+  (segment (start 101.092 118.259) (end 101.092 110.692) (width 0.254) (layer "F.Cu") (net 23))
   (segment (start 88.4915 119.38) (end 87.5155 118.404) (width 0.254) (layer "F.Cu") (net 23))
-  (segment (start 98.926 108.07) (end 97.358 108.07) (width 0.254) (layer "F.Cu") (net 23))
   (segment (start 91.948 119.38) (end 88.4915 119.38) (width 0.254) (layer "F.Cu") (net 23))
-  (segment (start 99.822 119.38) (end 101.092 118.11) (width 0.254) (layer "F.Cu") (net 23))
+  (segment (start 99.971 119.38) (end 101.092 118.259) (width 0.254) (layer "F.Cu") (net 23))
   (zone (net 0) (net_name "") (layer "F.Cu") (hatch edge 0.5)
     (connect_pads (clearance 0))
@@
         (xy 62.23 40.386)
         (xy 128.778 39.624)
-        (xy 122.682 137.16)
-        (xy 57.15 129.286)
+        (xy 123.282 147.06)
+        (xy 57.75 139.186)
       )
     )
